File: SD-interface.kicad_sch (KiCad schematic)
At the start: 18 parts, among them J8 SD_Card_Receptacle, U15 GL3224-OIY04, U16 TPD4E02B04DQA, U17 TPD4E02B04DQA, Y2 25MHz +-0.03%

Commit message: Design rule file added, lots of minor tweaks, routing done (including differential pairs), DRC done/
Parts:
- C70, C71, C72, C73, C76, C77: value 100nF -> 0.1uF; LCSC Part C181043 -> C181043
- C74, C75: LCSC Part C2980695 -> C2980695
- J8: Mouser Part No  179-SD-2-A -> 179-SD-2-A
- R59: LCSC Part C137858 -> C137858
Other:
- company: (none) -> Karol Woźniak
Changed lines of the file:
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@@
 	(title_block
 		(title "USB Hub")
+		(date "2026-03-18")
+		(company "Karol Woźniak")
 	)
 	(bus_alias "USB3"
@@
 		(polyline
 			(pts
+				(xy 137.16 35.56) (xy 137.16 41.91) (xy 144.78 41.91) (xy 144.78 35.56)
+			)
+			(stroke
+				(width 0)
+				(type dash)
+			)
+			(fill
+				(type none)
+			)
+		)
+	)
+	(rule_area
+		(polyline
+			(pts
 				(xy 53.34 34.29) (xy 53.34 50.8) (xy 86.36 50.8) (xy 86.36 34.29)
 			)
@@
 		(length 2.54)
 		(shape round)
+		(at 144.78 41.91 180)
+		(fields_autoplaced yes)
+		(effects
+			(font
+				(size 1.27 1.27)
+			)
+			(justify right bottom)
+		)
+		(property "Netclass" "USB_SS"
+			(at 145.4785 44.45 0)
+			(effects
+				(font
+					(size 1.27 1.27)
+				)
+				(justify left)
+			)
+		)
+		(property "Component Class" ""
+			(at 29.21 -45.72 0)
+			(effects
+				(font
+					(size 1.27 1.27)
+					(italic yes)
+				)
+			)
+		)
+	)
+	(netclass_flag ""
+		(length 2.54)
+		(shape round)
 		(at 62.23 50.8 180)
 		(fields_autoplaced yes)
@@
 			)
 		)
-		(property "Value" "100nF"
+		(property "Value" "0.1uF"
 			(at 20.828 59.944 0)
 			(effects
@@
 			)
 		)
-		(property "LCSC Part" "C181043 "
+		(property "LCSC Part" "C181043"
 			(at 20.32 57.15 0)
 			(effects
@@
 			)
 		)
-		(property "Mouser Part No " "179-SD-2-A "
+		(property "Mouser Part No " "179-SD-2-A"
 			(at 247.65 49.53 0)
 			(effects
@@
 			)
 		)
-		(property "Value" "100nF"
+		(property "Value" "0.1uF"
 			(at 48.768 80.01 0)
 			(effects
@@
 			)
 		)
-		(property "LCSC Part" "C181043 "
+		(property "LCSC Part" "C181043"
 			(at 48.26 77.47 0)
 			(effects
@@
 			)
 		)
-		(property "LCSC Part" "C2980695 "
+		(property "LCSC Part" "C2980695"
 			(at 78.74 40.64 90)
 			(effects
@@
 			)
 		)
-		(property "Value" "100nF"
+		(property "Value" "0.1uF"
 			(at 30.988 80.01 0)
 			(effects
@@
 			)
 		)
-		(property "LCSC Part" "C181043 "
+		(property "LCSC Part" "C181043"
 			(at 30.48 77.47 0)
 			(effects
@@
 			)
 		)
-		(property "LCSC Part" "C2980695 "
+		(property "LCSC Part" "C2980695"
 			(at 72.39 38.1 90)
 			(effects
@@
 			)
 		)
-		(property "Value" "100nF"
+		(property "Value" "0.1uF"
 			(at 39.878 80.01 0)
 			(effects
@@
 			)
 		)
-		(property "LCSC Part" "C181043 "
+		(property "LCSC Part" "C181043"
 			(at 39.37 77.47 0)
 			(effects
@@
 			)
 		)
-		(property "Value" "100nF"
+		(property "Value" "0.1uF"
 			(at 29.718 59.944 0)
 			(effects
@@
 			)
 		)
-		(property "LCSC Part" "C181043 "
+		(property "LCSC Part" "C181043"
 			(at 29.21 57.15 0)
 			(effects
@@
 			)
 		)
-		(property "Value" "100nF"
+		(property "Value" "0.1uF"
 			(at 22.098 80.01 0)
 			(effects
@@
 			)
 		)
-		(property "LCSC Part" "C181043 "
+		(property "LCSC Part" "C181043"
 			(at 20.32 77.47 0)
 			(effects
@@
 			)
 		)
-		(property "LCSC Part" "C137858 "
+		(property "LCSC Part" "C137858"
 			(at 74.93 111.76 90)
 			(effects
