File: USB-A1.kicad_sch (KiCad schematic)
At the start: 23 parts, among them J10 USB3_A, J9 USB3_A, U18 UCS2114-1-V/G4, U19 TPD4E02B04DQA, U20 TPD4E02B04DQA, U32 TPD4E02B04DQA

Commit message: Design rule file added, lots of minor tweaks, routing done (including differential pairs), DRC done/
Parts:
- added R100, R101: 10k, Resistor_SMD:R_0402_1005Metric, symbol Device:R
- added R102: 0, Resistor_SMD:R_0603_1608Metric, symbol Device:R
- added U32: TPD4E02B04DQA, Package_SON:USON-10_2.5x1.0mm_P0.5mm, symbol Snapeda:TPD4E02B04DQA
- C84: LCSC Part C181043 -> C181043
- J10, J9: LCSC Part C5119948 -> C5429469
- R64, R65: LCSC Part C327253 -> C327253
- TP5, TP6: now left out of the parts list
- U18: value UCS2114-1-V/G4 -> UCS2113; Mouser Part No  579-UCS2114-1-V/LX -> (none)
- renumbered U32 to U33
Connections:
- net +5V_USB_A: now also R100.2, R101.2, R102.1; no longer U18.13 (COMM_ILIM)
- net GND: now also J10.MH1 (SHIELD), J10.MH4 (SHIELD), J9.MH1 (SHIELD), J9.MH2 (SHIELD), J9.MH3 (SHIELD), J9.MH4 (SHIELD), U32.3 (G), U32.8 (G); no longer J10.10 (SHIELD), J9.10 (SHIELD)
- net USB-A1.D+: now also U32.5 (IO4), U32.6 (NC); no longer U33.1 (IO1), U33.10 (NC)
- net USB-A1.D-: now also U32.4 (IO3), U32.7 (NC); no longer U33.2 (IO2), U33.9 (NC)
- net USB-A2.D+: now also U33.4 (IO3), U33.7 (NC); no longer U33.5 (IO4), U33.6 (NC)
- net USB-A2.D-: now also U33.5 (IO4), U33.6 (NC); no longer U33.4 (IO3), U33.7 (NC)
- net at R62.1, U18.16 (ALERT#2): now also R101.1
- net at R61.1, U18.20 (ALERT#1): now also R100.1
- new net: U33.1 (IO1), U33.10 (NC)
- new net: U33.2 (IO2), U33.9 (NC)
- new net: U32.1 (IO1), U32.10 (NC)
- new net: U32.2 (IO2), U32.9 (NC)
- new net COMM_ILIM: R102.2, U18.13 (COMM_ILIM)
Other:
- company: (none) -> Karol Woźniak
- moved on the sheet: J10, J9, R62, R63
