File: USB-C1.kicad_sch (KiCad schematic)
At the start: 32 parts, among them J2 USB_C_Receptacle, J3 I2C_HD3SS3220, U3 HD3SS3220IRNHR, U4 TPS2068EDBVR, U5 TPD4E02B04DQA, U6 TPD4E02B04DQA, U7 TPD4E02B04DQA

Commit message: Design rule file added, lots of minor tweaks, routing done (including differential pairs), DRC done/
Parts:
- C23: value 100uF -> 100uF (6.3V); LCSC Part C141660 -> C141660
- C24, C25, C26, C27, C28: value 100nF -> 0.1uF; LCSC Part C181043 -> C181043
- C30: LCSC Part C181043 -> C181043
- J2: Mouser Part No  640-USB4200-03-A -> 640-USB4200-03-A
- J3, JP1, TP1, TP2: now left out of the parts list
- R11: Mouser Part No  603-RT1206CRE07900KL -> 603-RT1206CRE07900KL
- R12, R13: LCSC Part C25764 -> C25764
- R15: LCSC Part C2902631 -> C2902631
- R17: LCSC Part C5948099 -> C5948099
- R19: LCSC Part C327253 -> C327253
Connections:
- net GND: now also J2.MH1 (SHIELD), J2.MH2 (SHIELD), J2.MH3 (SHIELD), J2.MH4 (SHIELD); no longer J2.S1 (SHIELD)
- net USB3_IN.RX1+: now also U3.10 (RXN); no longer U3.9 (RXP)
- net USB3_IN.RX1-: now also U3.9 (RXP); no longer U3.10 (RXN)
- net USB3_IN.TX1+: now also U3.7 (TXN); no longer U3.6 (TXP)
- net USB3_IN.TX1-: now also U3.6 (TXP); no longer U3.7 (TXN)
Other:
- company: (none) -> Karol Woźniak
Changed lines of the file:
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@@
 	(title_block
 		(title "USB Hub")
+		(date "2026-03-18")
+		(company "Karol Woźniak")
 	)
 	(rectangle
@@
 		)
 	)
+	(label "USB3_IN.TX1+"
+		(at 49.53 86.36 0)
+		(effects
+			(font
+				(size 1.27 1.27)
+			)
+			(justify left bottom)
+		)
+	)
 	(label "I2C_HD3SS3220.SDA"
 		(at 46.99 76.2 0)
@@
 		)
 	)
-	(label "USB3_IN.RX1-"
-		(at 48.26 93.98 0)
+	(label "USB-C1.CC1"
+		(at 128.27 40.64 0)
 		(effects
 			(font
@@
 		)
 	)
-	(label "USB-C1.CC1"
-		(at 128.27 40.64 0)
+	(label "USB-C1.TX2+"
+		(at 218.44 73.66 0)
 		(effects
 			(font
@@
 		)
 	)
-	(label "USB-C1.TX2+"
-		(at 218.44 73.66 0)
+	(label "USB3_IN.RX1-"
+		(at 49.53 91.44 0)
 		(effects
 			(font
@@
 		)
 	)
-	(label "USB3_IN.RX1+"
-		(at 48.26 91.44 0)
-		(effects
-			(font
-				(size 1.27 1.27)
-			)
-			(justify left bottom)
-		)
-	)
-	(label "USB3_IN.TX1+"
-		(at 48.26 83.82 0)
-		(effects
-			(font
-				(size 1.27 1.27)
-			)
-			(justify left bottom)
-		)
-	)
 	(label "USB3_IN{USB3}"
 		(at 204.47 35.56 0)
@@
 		)
 	)
+	(label "USB3_IN.TX1-"
+		(at 49.53 83.82 0)
+		(effects
+			(font
+				(size 1.27 1.27)
+			)
+			(justify left bottom)
+		)
+	)
 	(label "ID"
 		(at 39.37 134.62 0)
@@
 		)
 	)
-	(label "VCONN_FAULT_N"
-		(at 52.07 68.58 0)
+	(label "USB3_IN.RX1+"
+		(at 49.53 93.98 0)
 		(effects
 			(font
@@
 		)
 	)
-	(label "USB-C1.TX2+"
-		(at 152.4 73.66 0)
+	(label "VCONN_FAULT_N"
+		(at 52.07 68.58 0)
 		(effects
 			(font
@@
 		)
 	)
-	(label "USB3_IN.TX1-"
-		(at 48.26 86.36 0)
+	(label "USB-C1.TX2+"
+		(at 152.4 73.66 0)
 		(effects
 			(font
@@
 		(polyline
 			(pts
+				(xy 217.17 38.1) (xy 217.17 44.45) (xy 233.68 44.45) (xy 233.68 38.1)
+			)
+			(stroke
+				(width 0)
+				(type dash)
+			)
+			(fill
+				(type none)
+			)
+		)
+	)
+	(rule_area
+		(polyline
+			(pts
 				(xy 48.26 80.01) (xy 48.26 97.79) (xy 66.04 97.79) (xy 66.04 80.01)
 			)
@@
 		(length 2.54)
 		(shape round)
+		(at 224.79 44.45 180)
+		(fields_autoplaced yes)
+		(effects
+			(font
+				(size 1.27 1.27)
+			)
+			(justify right bottom)
+		)
+		(property "Netclass" "USB_SS"
+			(at 225.4885 46.99 0)
+			(effects
+				(font
+					(size 1.27 1.27)
+				)
+				(justify left)
+			)
+		)
+		(property "Component Class" ""
+			(at 109.22 -43.18 0)
+			(effects
+				(font
+					(size 1.27 1.27)
+					(italic yes)
+				)
+			)
+		)
+	)
+	(netclass_flag ""
+		(length 2.54)
+		(shape round)
 		(at 57.15 97.79 180)
 		(fields_autoplaced yes)
@@
 			)
 		)
-		(property "Value" "100nF"
+		(property "Value" "0.1uF"
 			(at 141.224 59.944 90)
 			(effects
@@
 			)
 		)
-		(property "LCSC Part" "C181043 "
+		(property "LCSC Part" "C181043"
 			(at 137.16 60.96 90)
 			(effects
@@
 			)
 		)
-		(property "Mouser Part No " "603-RT1206CRE07900KL "
+		(property "Mouser Part No " "603-RT1206CRE07900KL"
 			(at 48.26 45.72 0)
 			(effects
@@
 		(unit 1)
 		(exclude_from_sim no)
-		(in_bom yes)
+		(in_bom no)
 		(on_board yes)
 		(dnp no)
@@
 		(unit 1)
 		(exclude_from_sim no)
-		(in_bom yes)
+		(in_bom no)
 		(on_board yes)
 		(dnp no)
@@
 			)
 		)
-		(property "Value" "100nF"
+		(property "Value" "0.1uF"
 			(at 147.574 62.484 90)
 			(effects
@@
 			)
 		)
-		(property "LCSC Part" "C181043 "
+		(property "LCSC Part" "C181043"
 			(at 143.51 63.5 90)
 			(effects
@@
 			)
 		)
-		(property "LCSC Part" "C25764 "
+		(property "LCSC Part" "C25764"
 			(at 43.18 55.88 90)
 			(effects
@@
 		(unit 1)
 		(exclude_from_sim no)
-		(in_bom yes)
+		(in_bom no)
 		(on_board yes)
 		(dnp no)
@@
 			)
 		)
-		(property "LCSC Part" "C181043 "
+		(property "LCSC Part" "C181043"
 			(at 36.83 133.35 0)
 			(effects
@@
 		(unit 1)
 		(exclude_from_sim no)
-		(in_bom yes)
+		(in_bom no)
 		(on_board yes)
 		(dnp no)
@@
 			)
 		)
-		(property "LCSC Part" "C327253 "
+		(property "LCSC Part" "C327253"
 			(at 118.11 170.18 0)
 			(effects
@@
 			)
 		)
-		(property "LCSC Part" "C2902631 "
+		(property "LCSC Part" "C2902631"
 			(at 49.53 71.12 90)
 			(effects
@@
 			)
 		)
-		(property "LCSC Part" "C5948099 "
+		(property "LCSC Part" "C5948099"
 			(at 121.92 133.35 90)
 			(effects
@@
 			)
 		)
-		(property "Mouser Part No " "640-USB4200-03-A "
+		(property "Mouser Part No " "640-USB4200-03-A"
 			(at 248.92 50.8 0)
 			(effects
@@
 		(pin "A6"
 		)
-		(pin "S1"
+		(pin "MH3"
 		)
 		(pin "B4"
@@
 		(pin "B3"
 		)
+		(pin "MH4"
+		)
+		(pin "MH2"
+		)
+		(pin "MH1"
+		)
 		(instances
 			(project ""
@@
 			)
 		)
-		(property "Value" "100nF"
+		(property "Value" "0.1uF"
 			(at 147.574 75.184 90)
 			(effects
@@
 			)
 		)
-		(property "LCSC Part" "C181043 "
+		(property "LCSC Part" "C181043"
 			(at 143.51 76.2 90)
 			(effects
@@
 			)
 		)
-		(property "Value" "100uF"
+		(property "Value" "100uF (6.3V)"
 			(at 24.13 31.7499 0)
 			(effects
@@
 			)
 		)
-		(property "LCSC Part" "C141660 "
+		(property "LCSC Part" "C141660"
 			(at 20.32 30.48 0)
 			(effects
@@
 			)
 		)
-		(property "Value" "100nF"
+		(property "Value" "0.1uF"
 			(at 36.83 31.7499 0)
 			(effects
@@
 			)
 		)
-		(property "LCSC Part" "C181043 "
+		(property "LCSC Part" "C181043"
 			(at 33.02 30.48 0)
 			(effects
@@
 			)
 		)
-		(property "LCSC Part" "C25764 "
+		(property "LCSC Part" "C25764"
 			(at 52.07 60.96 90)
 			(effects
@@
 			)
 		)
-		(property "Value" "100nF"
+		(property "Value" "0.1uF"
 			(at 141.224 72.644 90)
 			(effects
@@
 			)
 		)
-		(property "LCSC Part" "C181043 "
+		(property "LCSC Part" "C181043"
 			(at 137.16 73.66 90)
 			(effects
