File: USB-C2.kicad_sch (KiCad schematic)
At the start: 92 parts, among them J4 USB_C_Receptacle, J5 I2C2_PD_Controller, J6 I2C_Mux, J7 I2C_EEPROM, SW2 FW_Upgrade, U10 24LC256, U11 TPD4E02B04DQA, U12 TPD4E02B04DQA, U13 TPD4E02B04DQA, U14 TUSB1142IRNQR_C5216209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

Commit message: Design rule file added, lots of minor tweaks, routing done (including differential pairs), DRC done/
Parts:
- C32, C34: value 4.7uF 6.3V -> 4.7uF 10V; LCSC Part C6119944 -> C318563
- C33, C35, C37, C39, C40, C56: LCSC Part C181043 -> C181043
- C36: LCSC Part C6119944 -> C318563
- C38: footprint Capacitor_SMD:C_1812_4532Metric -> Capacitor_SMD:C_1206_3216Metric; LCSC Part C141660 -> C309062
- C41, C43, C46: LCSC Part C114401 -> C307445
- C45: value 0.1uF 40V -> 0.1uF (50V)
- C50: Mouser Part No  710-865080645010 -> 710-865080645010
- C51: footprint Capacitor_THT:C_Radial_D6.3mm_H11.0mm_P2.50mm -> Capacitor_SMD:CP_Elec_6.3x7.7; LCSC Part C109392 -> C311622
- C66, C67, C68, C69: value 100nF -> 0.1uF; LCSC Part C181043 -> C181043
- J4: Mouser Part No  640-USB4200-03-A -> 640-USB4200-03-A
- J5, J6, J7, TP3, TP4: now left out of the parts list
- R21, R22, R25, R26: LCSC Part C966185 -> C966185
- R27, R31: value 10 (0.1W) -> 10 (0.25W)
- R28: LCSC Part C332644 -> C407669; Mouser Part No  71-CRCW04026R65FKEDH -> (none)
- R30: LCSC Part C93945 -> C93945
- R34, R40, R43, R50: LCSC Part C11702 -> C11702
- R41, R42, R44, R47, R48, R49, R52, R53: LCSC Part C469665 -> C166074
- SW2: LCSC Part C913788 -> C913788
- U9: Mouser Part No  595-TPS25762CQRQLRQ1 -> (none)
Connections:
- net PGND: now also J4.MH1 (SHIELD), J4.MH2 (SHIELD), J4.MH3 (SHIELD), J4.MH4 (SHIELD); no longer J4.S1 (SHIELD)
- net CSP: now reaches C46.2, R31.1, U9.28 (CSP)
- net CS_1P: now reaches C48.1, C49.1, C50.1, R31.2, R32.2, U9.11 (OUT)
- net CTX1_R+: now reaches C59.2, R48.1
- net CTX1_R-: now reaches C60.2, R49.1
- net CTX2_R+: now reaches C57.2, R41.1
- net CSN: now reaches C46.1, R27.1, U9.29 (CSN/BUS)
- net CTX2_R-: now reaches C58.2, R42.1
Other:
- note removed: "CHECK FOOTPRINT"
- company: (none) -> Karol Woźniak
- moved on the sheet: R41, R42, R44, R47, R48, R49, R52, R53
