File: USB-E_UP.kicad_sch (KiCad schematic)
At the start: 5 parts, among them J14 USB_C_Internal_Connector, U30 TPD4E02B04DQA, U31 TPD4E02B04DQA

Commit message: Design rule file added, lots of minor tweaks, routing done (including differential pairs), DRC done/
Other:
- company: (none) -> Karol Woźniak
Changed lines of the file:
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@@
 	(title_block
 		(title "USB Hub")
+		(date "2026-03-18")
+		(company "Karol Woźniak")
 	)
 	(rectangle
