File: USB7206C.kicad_sch (KiCad schematic)
At the start: 42 parts, among them J1 USB_SPI_(Opt), SW1 RESET_HUB, U1 USB7206C/KDX, U2 MIC803-29D4VM3-TR, Y1 25MHz

Commit message: Design rule file added, lots of minor tweaks, routing done (including differential pairs), DRC done/
Parts:
- added R103: 200k, Resistor_SMD:R_0402_1005Metric, symbol Device:R
- added R104: 10, Resistor_SMD:R_0603_1608Metric, symbol Device:R
- C1, C11, C12, C13, C14, C15, C16, C17, C18, C2, C3, C4, C5, C6, C7, C8, C9: LCSC Part C181043 -> C181043
- C10, C19: value 4.7uF -> 4.7uF 10V; footprint Capacitor_SMD:C_0805_2012Metric -> Capacitor_SMD:C_0402_1005Metric; LCSC Part C6119944 -> C318563
- C127, C128, C129, C130: value 100nF -> 0.1uF; LCSC Part C181043 -> C181043
- J1: footprint Connector_PinHeader_1.00mm:PinHeader_1x03_P1.00mm_Vertical -> Connector_PinHeader_1.00mm:PinHeader_1x07_P1.00mm_Vertical; now left out of the parts list
- R1: LCSC Part C102781 -> C102781
- R10, R9: LCSC Part C25764 -> C25764
- R5: LCSC Part C25779 -> C25779
- R8: LCSC Part C25741 -> C25741
- SW1: LCSC Part C913788 -> C913788
- U1: Mouser Part No  579-USB7206C/KDX -> 579-USB7206C/KDX
- Y1: value 25MHz -> 25MHz +-0.03%
Connections:
- net CFG_BC_EN: now also R104.1
- net CFG_NON_REM: now also R103.1
- net GND: now also R103.2, R104.2
- net USB3_DN1.TX1+: no longer U1.8 (USB3DN_TXDM1)
- new net USB3_DN1.TX1-: U1.8 (USB3DN_TXDM1)
Other:
- company: (none) -> Karol Woźniak
