File: USB_hub.kicad_sch (KiCad schematic)
At the start: 0 parts

Commit message: Design rule file added, lots of minor tweaks, routing done (including differential pairs), DRC done/
Other:
- company: (none) -> Karol Woźniak
Changed lines of the file:
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@@
 	(title_block
 		(title "USB Hub")
+		(date "2026-03-18")
+		(company "Karol Woźniak")
 	)
 	(text "these connections may change for better routing "
@@
 		)
 	)
+	(bus_entry
+		(at 91.44 57.15)
+		(size 2.54 2.54)
+		(stroke
+			(width 0)
+			(type default)
+		)
+	)
